Commit message: 24/09/29 normal updates

File: src/chapt6/robot_description/urdf/b_class_car/base.urdf.xacro (robot description, xacro)
@@ -255,28 +255,33 @@
         <material>Gazebo/Black</material>
     </gazebo>
+    <ros2_control name="CarControlSystem" type="system">
+      <hardware>
+        <plugin>ros2_control_demo_hardware/CarHardware</plugin>
+        <param name="example_param_write_for_sec">0.01</param>
+        <param name="example_param_read_for_sec">0.01</param>
+      </hardware>
+      <!-- 控制后轮驱动 -->
+      <joint name="rear_right_wheel_joint">
+        <command_interface name="velocity"/>
+        <state_interface name="velocity"/>
+      </joint>
+      <joint name="rear_left_wheel_joint">
+        <command_interface name="velocity"/>
+        <state_interface name="velocity"/>
+      </joint>
+      <!-- 控制前轮转向 -->
+      <joint name="front_right_steering_joint">
+        <command_interface name="position"/>
+        <state_interface name="position"/>
+      </joint>
+      <joint name="front_left_steering_joint">
+        <command_interface name="position"/>
+        <state_interface name="position"/>
+      </joint>
+    </ros2_control>
     <gazebo>
-            <plugin name='diff_drive' filename='libgazebo_ros_diff_drive.so'>
-                <ros>
-                    <namespace>/</namespace>
-                    <remapping>cmd_vel:=cmd_vel</remapping>
-                    <remapping>odom:=odom</remapping>
-                </ros>
-                <update_rate>30</update_rate>
-                <!-- wheels -->
-                <left_joint>left_wheel_joint</left_joint>
-                <right_joint>right_wheel_joint</right_joint>
-                <!-- kinematics -->
-                <wheel_separation>0.2</wheel_separation>
-                <wheel_diameter>0.064</wheel_diameter>
-                <!-- limits -->
-                <max_wheel_torque>20</max_wheel_torque>
-                <max_wheel_acceleration>1.0</max_wheel_acceleration>
-                <!-- output -->
-                <publish_odom>true</publish_odom>
-                <publish_odom_tf>true</publish_odom_tf>
-                <publish_wheel_tf>true</publish_wheel_tf>
-                <odometry_frame>odom</odometry_frame>
-                <robot_base_frame>base_footprint</robot_base_frame>
-            </plugin>
+      <plugin filename="libgazebo_ros2_control.so" name="gazebo_ros2_control">
+        <param>$(find robot_desscription)/config/controllers.yaml</param>
+      </plugin>
     </gazebo>
 </robot>

Commit message: 24/11/28 normal update_1

File: src/chapt6/robot_description/urdf/b_class_car/base.urdf.xacro (robot description, xacro)
@@ -1,3 +1,3 @@
-<robot name="classb_car" xmlns:xacro="http://www.ros.org/wiki/xacro">
+<robot name="classb_car" xmlns:xacro="http://www.ros.org/wiki/xacro">       <!-- 表示urdf使用xacro宏语言 -->
     <xacro:property name="PI" value="3.141"/>
     <xacro:property name="base_length" value="2.695"/>
@@ -252,5 +252,5 @@
       <dynamics damping="0.1"/>
     </joint>
-    <gazebo reference="base_link">
+    <gazebo reference="base_link">               <!-- 设置base)link在gazebo世界中的颜色为黑色 -->
         <material>Gazebo/Black</material>
     </gazebo>

File: src/chapt6/robot_description/urdf/b_class_car/sensor/imu.urdf.xacro (robot description, xacro)
@@ -1,5 +1,5 @@
 <?xml version="1.0"?>
 <robot xmlns:xacro="http://www.ros.org/wiki/xacro">
-    <xacro:macro name="imu_xacro" params="xyz">
+    <xacro:macro name="imu_xacro" params="xyz">                     <!-- 定义IMU传感器 -->
         <link name="imu_link">
             <visual>
